Commit message: Fixed pose goal for the moveit_interface package such that the arms can actually achieve the desired pose. Updated end-effector location to be between gripper fingers in Moveit also (instead of the end of the arm). Fixed bug in launch file

File: interbotix_ros_xslocobots/interbotix_xslocobot_moveit/config/srdf/locobot_px100.srdf.xacro (robot description, xacro)
@@ -21,9 +21,9 @@
         <joint name="wrist_angle" />
         <joint name="ee_arm" />
+        <joint name="gripper_bar" />
+        <joint name="ee_bar" />
+        <joint name="ee_gripper" />
     </group>
     <group name="interbotix_gripper">
-        <link name="$(arg robot_name)/gripper_bar_link" />
-        <link name="$(arg robot_name)/fingers_link" />
-        <link name="$(arg robot_name)/ee_gripper_link" />
         <link name="$(arg robot_name)/left_finger_link" />
         <link name="$(arg robot_name)/right_finger_link" />
@@ -61,5 +61,5 @@
     </group_state>
     <!--END EFFECTOR: Purpose: Represent information about an end effector.-->
-    <end_effector name="interbotix_gripper" parent_link="$(arg robot_name)/ee_arm_link" group="interbotix_gripper" />
+    <end_effector name="interbotix_gripper" parent_link="$(arg robot_name)/ee_gripper_link" group="interbotix_gripper" />
     <!--DISABLE COLLISIONS: By default it is assumed that any link of the robot could potentially come into collision with any other link in the robot. This tag disables collision checking between a specified pair of links. -->
     <disable_collisions link1="$(arg robot_name)/ar_tag_link" link2="$(arg robot_name)/caster_back_link" reason="Never" />

File: interbotix_ros_xslocobots/interbotix_xslocobot_moveit/config/srdf/locobot_wx200.srdf.xacro (robot description, xacro)
@@ -22,9 +22,9 @@
         <joint name="wrist_rotate" />
         <joint name="ee_arm" />
+        <joint name="gripper_bar" />
+        <joint name="ee_bar" />
+        <joint name="ee_gripper" />
     </group>
     <group name="interbotix_gripper">
-        <link name="$(arg robot_name)/gripper_bar_link" />
-        <link name="$(arg robot_name)/fingers_link" />
-        <link name="$(arg robot_name)/ee_gripper_link" />
         <link name="$(arg robot_name)/left_finger_link" />
         <link name="$(arg robot_name)/right_finger_link" />
@@ -65,5 +65,5 @@
     </group_state>
     <!--END EFFECTOR: Purpose: Represent information about an end effector.-->
-    <end_effector name="interbotix_gripper" parent_link="$(arg robot_name)/ee_arm_link" group="interbotix_gripper" />
+    <end_effector name="interbotix_gripper" parent_link="$(arg robot_name)/ee_gripper_link" group="interbotix_gripper" />
     <!--DISABLE COLLISIONS: By default it is assumed that any link of the robot could potentially come into collision with any other link in the robot. This tag disables collision checking between a specified pair of links. -->
     <disable_collisions link1="$(arg robot_name)/ar_tag_link" link2="$(arg robot_name)/forearm_link" reason="Never" />

File: interbotix_ros_xslocobots/interbotix_xslocobot_moveit/config/srdf/locobot_wx250s.srdf.xacro (robot description, xacro)
@@ -23,9 +23,9 @@
         <joint name="wrist_rotate" />
         <joint name="ee_arm" />
+        <joint name="gripper_bar" />
+        <joint name="ee_bar" />
+        <joint name="ee_gripper" />
     </group>
     <group name="interbotix_gripper">
-        <link name="$(arg robot_name)/gripper_bar_link" />
-        <link name="$(arg robot_name)/fingers_link" />
-        <link name="$(arg robot_name)/ee_gripper_link" />
         <link name="$(arg robot_name)/left_finger_link" />
         <link name="$(arg robot_name)/right_finger_link" />
@@ -69,5 +69,5 @@
     </group_state>
     <!--END EFFECTOR: Purpose: Represent information about an end effector.-->
-    <end_effector name="interbotix_gripper" parent_link="$(arg robot_name)/ee_arm_link" group="interbotix_gripper" />
+    <end_effector name="interbotix_gripper" parent_link="$(arg robot_name)/ee_gripper_link" group="interbotix_gripper" />
     <!--DISABLE COLLISIONS: By default it is assumed that any link of the robot could potentially come into collision with any other link in the robot. This tag disables collision checking between a specified pair of links. -->
     <disable_collisions link1="$(arg robot_name)/ar_tag_link" link2="$(arg robot_name)/gripper_bar_link" reason="Default" />
