Commit message: update some incorrect min/max position limits for the motors. also get rid of unnessary picture in the ros_control package.

File: interbotix_ros_xslocobots/interbotix_xslocobot_descriptions/urdf/mobile_px100.urdf.xacro (robot description, xacro)
@@ -140,5 +140,5 @@
   <joint name="wrist_angle" type="revolute">
     <axis xyz="0 1 0"/>
-    <limit effort="1" lower="${radians(-123)}" upper="${radians(100)}"  velocity="${pi}"/>
+    <limit effort="1" lower="${radians(-100)}" upper="${radians(123)}"  velocity="${pi}"/>
     <origin rpy="0 0 0" xyz="0.1 0 0"/>
     <parent link="$(arg robot_name)/forearm_link"/>
