Commit message: Adds the Perception Pipeline to allow the arms to pick up small objects found using a color/depth camera

File: interbotix_ros_xslocobots/interbotix_xslocobot_descriptions/urdf/locobot.urdf.xacro (robot description, xacro)
@@ -413,5 +413,5 @@
   </link>
   <joint name="camera" type="fixed">
-    <origin rpy="0 0 0" xyz="0.04198 0.0175 0.000009"/>
+    <origin rpy="0 0 0" xyz="0.05318 0.0175 0.000009"/>
     <parent link="$(arg robot_name)/tilt_link"/>
     <child link="$(arg robot_name)/camera_link"/>
@@ -434,5 +434,5 @@
     </collision>
     <inertial>
-      <origin rpy="0 0 0" xyz="0.0016276600 -0.0158176000 0.0000026190"/>
+      <origin rpy="0 0 0" xyz="-0.008972 -0.015818 0.000003"/>
       <mass value="0.072"/>
       <inertia ixx="0.0000465400" ixy="0.0000003028" ixz="0.0000000245" iyy="0.0000069128" iyz="0.0000000248" izz="0.0000468600"/>

Commit message: gpd mustard works

File: interbotix_ros_xslocobots/interbotix_xslocobot_descriptions/urdf/locobot.urdf.xacro (robot description, xacro)
@@ -447,4 +447,10 @@
     </inertial>
   </link>
+  <link name="$(arg robot_name)_camera_optical_link"/>
+  <joint name="$(arg robot_name)_camera_optical_joint" type="fixed">
+      <origin xyz="0 0 0" rpy="-${pi/2} 0 -${pi/2}"/>
+      <parent link="$(arg robot_name)_camera_link"/>
+      <child link="$(arg robot_name)_camera_optical_link"/>
+    </joint>
   <!-- ********************************** Lidar **********************************  -->
   <xacro:if value="$(arg show_lidar)">

File: interbotix_ros_xslocobots/interbotix_xslocobot_moveit/config/srdf/locobot_wx250s.srdf.xacro (robot description, xacro)
@@ -14,4 +14,7 @@
     <xacro:arg name="external_srdf_loc" default=""/>
     <xacro:property name="srdf_loc" value="$(arg external_srdf_loc)"/>
+    <group name="interbotix_neck">
+     <chain base_link="$(arg robot_name)_camera_tower_link" tip_link="$(arg robot_name)_camera_link"/>
+    </group>
     <group name="interbotix_arm">
      <chain base_link="$(arg robot_name)_arm_base_link" tip_link="$(arg robot_name)_gripper_bar_link"/>
@@ -33,4 +36,8 @@
         <link name="$(arg robot_name)_right_finger_link" />
     </group>
+    <group_state name="Home" group="interbotix_neck">
+        <joint name="tilt" value="0.8" />
+        <joint name="pan" value="0" />
+    </group_state>
     <!--GROUP STATES: Purpose: Define a named state for a particular group, in terms of joint values. This is useful to define states like 'folded arms'-->
     <group_state name="Home" group="interbotix_arm">

Commit message: [xslocobot_descriptions] Add Create3 descriptions
Add the Create3 to the locobot descripions. Other minor changes.

File: interbotix_ros_xslocobots/interbotix_xslocobot_descriptions/urdf/locobot.urdf.xacro (robot description, xacro)
@@ -3,4 +3,5 @@
   <xacro:arg name="arm_model" default=""/>
   <xacro:arg name="robot_model" default=""/>
+  <xacro:arg name="base_type" default=""/>
   <xacro:arg name="robot_name" default=""/>
   <xacro:arg name="show_lidar" default="true"/>
@@ -21,183 +22,492 @@
     <texture filename="package://interbotix_xslocobot_descriptions/meshes/interbotix_black.png"/>
   </material>
-    <!-- ********************************** Kobuki ********************************** -->
   <link name="$(arg robot_name)/base_footprint"/>
-  <joint name="base_joint" type="fixed">
-    <origin rpy="0 0 0" xyz="0 0 0.0102"/>
-    <parent link="$(arg robot_name)/base_footprint"/>
-    <child link="$(arg robot_name)/base_link"/>
-  </joint>
-  <link name="$(arg robot_name)/base_link">
-    <visual>
-      <origin rpy="0 0 0" xyz="0.001 0 0.05199"/>
-      <geometry>
-        <mesh filename="package://interbotix_xslocobot_descriptions/meshes/locobot_meshes/locobot_main_body.dae"/>
-      </geometry>
-    </visual>
-    <collision>
-      <origin rpy="0 0 0" xyz="0.0 0 0.05949"/>
-      <geometry>
-        <cylinder length="0.10938" radius="0.178"/>
-      </geometry>
-    </collision>
-    <inertial>
-      <origin rpy="0 0 0" xyz="0.01 0 0"/>
-      <mass value="2.4"/>
-      <inertia ixx="0.019995" ixy="0.0" ixz="0.0" iyy="0.019995" iyz="0.0" izz="0.03675"/>
-    </inertial>
-  </link>
-  <joint name="wheel_left_joint" type="continuous">
-    <axis xyz="0 0 1"/>
-    <origin rpy="-1.57079632679 0 0" xyz="0.00 0.115 0.0250"/>
-    <parent link="$(arg robot_name)/base_link"/>
-    <child link="$(arg robot_name)/wheel_left_link"/>
-  </joint>
-  <transmission name="trans_wheel_left_joint">
-    <type>transmission_interface/SimpleTransmission</type>
-    <joint name="wheel_left_joint">
-      <hardwareInterface>hardware_interface/EffortJointInterface</hardwareInterface>
-    </joint>
-    <actuator name="wheel_left_joint_motor">
-      <mechanicalReduction>1</mechanicalReduction>
-    </actuator>
-  </transmission>
-  <link name="$(arg robot_name)/wheel_left_link">
-    <visual>
+  <!-- ********************************** Kobuki ********************************** -->
+  <xacro:if value="${'$(arg base_type)' == 'kobuki'}">
+    <!-- Much of the following Kobuki description is taken from https://github.com/yujinrobot/kobuki/blob/23748ed3dfb082831ca8eaaef1a0b08588dbcb65/kobuki_description/urdf/kobuki.urdf.xacro -->
+    <!-- It has been modified to include the robot_name as a prefix to the links -->
+    <!-- The kobuki_description package is distributed under the 3-Clause BSD License, but no license file was found in the package. -->
+    <!-- The license from the kobuki_node package is given from https://github.com/yujinrobot/kobuki/blob/8f2fa7b9e5e98c503ba468602c3a5dd9be68fc26/kobuki_node/LICENSE below: -->
+    <!--
+      # Software License Agreement (BSD License)
+      #
+      # Copyright (c) 2012 Yujin Robot, Daniel Stonier, Jorge Santos,
+      # Marcus Liebhardt, Younghun Ju, Jihoon Lee
+      # All rights reserved.
+      #
+      # Redistribution and use in source and binary forms, with or without
+      # modification, are permitted provided that the following conditions
+      # are met:
+      #
+      #    * Redistributions of source code must retain the above copyright
+      #        notice, this list of conditions and the following disclaimer.
+      #    * Redistributions in binary form must reproduce the above
+      #        copyright notice, this list of conditions and the following
+      #        disclaimer in the documentation and/or other materials provided
+      #        with the distribution.
+      #    * Neither the name of Yujin Robot nor the names of its
+      #        contributors may be used to endorse or promote products derived
+      #        from this software without specific prior written permission.
+      #
+      # THIS SOFTWARE IS PROVIDED BY THE COPYRIGHT HOLDERS AND CONTRIBUTORS
+      # "AS IS" AND ANY EXPRESS OR IMPLIED WARRANTIES, INCLUDING, BUT NOT
+      # LIMITED TO, THE IMPLIED WARRANTIES OF MERCHANTABILITY AND FITNESS
+      # FOR A PARTICULAR PURPOSE ARE DISCLAIMED. IN NO EVENT SHALL THE
+      # COPYRIGHT OWNER OR CONTRIBUTORS BE LIABLE FOR ANY DIRECT, INDIRECT,
+      # INCIDENTAL, SPECIAL, EXEMPLARY, OR CONSEQUENTIAL DAMAGES (INCLUDING,
+      # BUT NOT LIMITED TO, PROCUREMENT OF SUBSTITUTE GOODS OR SERVICES;
+      # LOSS OF USE, DATA, OR PROFITS; OR BUSINESS INTERRUPTION) HOWEVER
+      # CAUSED AND ON ANY THEORY OF LIABILITY, WHETHER IN CONTRACT, STRICT
+      # LIABILITY, OR TORT (INCLUDING NEGLIGENCE OR OTHERWISE) ARISING IN
+      # ANY WAY OUT OF THE USE OF THIS SOFTWARE, EVEN IF ADVISED OF THE
+      # POSSIBILITY OF SUCH DAMAGE.
+    -->
+    <joint name="base_joint" type="fixed">
+      <origin rpy="0 0 0" xyz="0 0 0.0102"/>
+      <parent link="$(arg robot_name)/base_footprint"/>
+      <child link="$(arg robot_name)/base_link"/>
+    </joint>
+    <link name="$(arg robot_name)/base_link">
+      <visual>
+        <origin rpy="0 0 0" xyz="0.001 0 0.05199"/>
+        <geometry>
+          <mesh filename="package://interbotix_xslocobot_descriptions/meshes/locobot_meshes/locobot_main_body.dae"/>
+        </geometry>
+      </visual>
+      <collision>
+        <origin rpy="0 0 0" xyz="0.0 0 0.05949"/>
+        <geometry>
+          <cylinder length="0.10938" radius="0.178"/>
+        </geometry>
+      </collision>
+      <inertial>
+        <origin rpy="0 0 0" xyz="0.01 0 0"/>
+        <mass value="2.4"/>
+        <inertia ixx="0.019995" ixy="0.0" ixz="0.0" iyy="0.019995" iyz="0.0" izz="0.03675"/>
+      </inertial>
+    </link>
+    <joint name="wheel_left_joint" type="continuous">
+      <axis xyz="0 0 1"/>
+      <origin rpy="-1.57079632679 0 0" xyz="0.00 0.115 0.0250"/>
+      <parent link="$(arg robot_name)/base_link"/>
+      <child link="$(arg robot_name)/wheel_left_link"/>
+    </joint>
+    <transmission name="trans_wheel_left_joint">
+      <type>transmission_interface/SimpleTransmission</type>
+      <joint name="wheel_left_joint">
+        <hardwareInterface>hardware_interface/EffortJointInterface</hardwareInterface>
+      </joint>
+      <actuator name="wheel_left_joint_motor">
+        <mechanicalReduction>1</mechanicalReduction>
+      </actuator>
+    </transmission>
+    <link name="$(arg robot_name)/wheel_left_link">
+      <visual>
+        <origin rpy="0 0 0" xyz="0 0 0"/>
+        <geometry>
+          <mesh filename="package://interbotix_xslocobot_descriptions/meshes/locobot_meshes/locobot_wheel.dae"/>
+        </geometry>
+      </visual>
+      <collision>
+        <geometry>
+          <cylinder length="0.0206" radius="0.0352"/>
+        </geometry>
+          <origin rpy="0 0 0" xyz="0 0 0"/>
+      </collision>
+      <inertial>
+        <origin xyz="0 0 0"/>
+        <mass value="0.01"/>
+        <inertia ixx="0.001" ixy="0.0" ixz="0.0" iyy="0.001" iyz="0.0" izz="0.001"/>
+      </inertial>
+    </link>
+    <joint name="wheel_right_joint" type="continuous">
+      <axis xyz="0 0 1"/>
+      <origin rpy="-1.57079632679 0 0" xyz="0.00 -0.115 0.0250"/>
+      <parent link="$(arg robot_name)/base_link"/>
+      <child link="$(arg robot_name)/wheel_right_link"/>
+    </joint>
+    <transmission name="trans_wheel_right_joint">
+      <type>transmission_interface/SimpleTransmission</type>
+      <joint name="wheel_right_joint">
+        <hardwareInterface>hardware_interface/EffortJointInterface</hardwareInterface>
+      </joint>
+      <actuator name="wheel_right_joint_motor">
+        <mechanicalReduction>1</mechanicalReduction>
+      </actuator>
+    </transmission>
+    <link name="$(arg robot_name)/wheel_right_link">
+      <visual>
+        <origin rpy="0 0 0" xyz="0 0 0"/>
+        <geometry>
+          <mesh filename="package://interbotix_xslocobot_descriptions/meshes/locobot_meshes/locobot_wheel.dae"/>
+        </geometry>
+      </visual>
+      <collision>
+        <origin rpy="0 0 0" xyz="0 0 0"/>
+        <geometry>
+          <cylinder length="0.0206" radius="0.0350"/>
+        </geometry>
+      </collision>
+      <inertial>
+        <origin xyz="0 0 0"/>
+        <mass value="0.01"/>
+        <inertia ixx="0.001" ixy="0.0" ixz="0.0" iyy="0.001" iyz="0.0" izz="0.001"/>
+      </inertial>
+    </link>
+    <joint name="caster_front_joint" type="fixed">
+      <origin rpy="-1.57079632679 0 0" xyz="0.115 0.0 0.007"/>
+      <parent link="$(arg robot_name)/base_link"/>
+      <child link="$(arg robot_name)/caster_front_link"/>
+    </joint>
+    <link name="$(arg robot_name)/caster_front_link">
+      <collision>
+        <origin rpy="0 0 0" xyz="0 0 0"/>
+        <geometry>
+          <cylinder length="0.0176" radius="0.017"/>
+        </geometry>
+      </collision>
+      <inertial>
+        <origin xyz="0 0 0"/>
+        <mass value="0.01"/>
+        <inertia ixx="0.001" ixy="0.0" ixz="0.0" iyy="0.001" iyz="0.0" izz="0.001"/>
+      </inertial>
+    </link>
+    <joint name="caster_back_joint" type="fixed">
+      <origin rpy="-1.57079632679 0 0" xyz="-0.135 0.0 0.009"/>
+      <parent link="$(arg robot_name)/base_link"/>
+      <child link="$(arg robot_name)/caster_back_link"/>
+    </joint>
+    <link name="$(arg robot_name)/caster_back_link">
+      <collision>
+        <origin rpy="0 0 0" xyz="0 0 0"/>
+        <geometry>
+          <cylinder length="0.0176" radius="0.017"/>
+        </geometry>
+      </collision>
+      <inertial>
+        <origin xyz="0 0 0"/>
+        <mass value="0.01"/>
+        <inertia ixx="0.001" ixy="0.0" ixz="0.0" iyy="0.001" iyz="0.0" izz="0.001"/>
+      </inertial>
+    </link>
+    <joint name="gyro_joint" type="fixed">
+      <origin rpy="0 0 0" xyz="0.056 0.062 0.0202"/>
+      <parent link="$(arg robot_name)/base_link"/>
+      <child link="$(arg robot_name)/gyro_link"/>
+    </joint>
+    <link name="$(arg robot_name)/gyro_link">
+      <inertial>
+        <origin rpy="0 0 0" xyz="0 0 0"/>
+        <mass value="0.001"/>
+        <inertia ixx="0.0001" ixy="0" ixz="0" iyy="0.000001" iyz="0" izz="0.0001"/>
+      </inertial>
+    </link>
+    <joint name="cliff_sensor_left_joint" type="fixed">
+      <origin rpy="0 1.57079632679 0" xyz="0.08734 0.13601 0.0214"/>
+      <parent link="$(arg robot_name)/base_link"/>
+      <child link="$(arg robot_name)/cliff_sensor_left_link"/>
+    </joint>
+    <link name="$(arg robot_name)/cliff_sensor_left_link">
+      <inertial>
+        <mass value="0.0001"/>
+        <origin xyz="0 0 0"/>
+        <inertia ixx="0.0001" ixy="0.0" ixz="0.0" iyy="0.0001" iyz="0.0" izz="0.0001"/>
+      </inertial>
+    </link>
+    <joint name="cliff_sensor_right_joint" type="fixed">
+      <origin rpy="0 1.57079632679 0" xyz="0.085 -0.13601 0.0214"/>
+      <parent link="$(arg robot_name)/base_link"/>
+      <child link="$(arg robot_name)/cliff_sensor_right_link"/>
+    </joint>
+    <link name="$(arg robot_name)/cliff_sensor_right_link">
+      <inertial>
+        <origin xyz="0 0 0"/>
+        <mass value="0.0001"/>
+        <inertia ixx="0.0001" ixy="0.0" ixz="0.0" iyy="0.0001" iyz="0.0" izz="0.0001"/>
+      </inertial>
+    </link>
+    <joint name="cliff_sensor_front_joint" type="fixed">
+      <origin rpy="0 1.57079632679 0" xyz="0.156 0.00 0.0214"/>
+      <parent link="$(arg robot_name)/base_link"/>
+      <child link="$(arg robot_name)/cliff_sensor_front_link"/>
+    </joint>
+    <link name="$(arg robot_name)/cliff_sensor_front_link">
+      <inertial>
+        <mass value="0.0001"/>
+        <origin xyz="0 0 0"/>
+        <inertia ixx="0.0001" ixy="0.0" ixz="0.0" iyy="0.0001" iyz="0.0" izz="0.0001"/>
+      </inertial>
+    </link>
+  </xacro:if> <!-- kobuki -->
+  <!-- ************************************* iRobot Create3 ************************************* -->
+  <xacro:if value="${'$(arg base_type)' == 'create3'}">
+    <!-- Much of the following iRobot Create3 description is taken from https://github.com/iRobotEducation/create3_sim/tree/6b8a4a6ce0d0902a7de117c29cbe55bfc52a4e54/irobot_create_common/irobot_create_description/urdf -->
+    <!-- The original 3-Clause BSD License is retained below -->
+    <!--
+      Copyright 2021 iRobot Corporation.
+      Redistribution and use in source and binary forms, with or without modification, are permitted provided that the following conditions are met:
+      1. Redistributions of source code must retain the above copyright notice, this list of conditions and the following disclaimer.
+      2. Redistributions in binary form must reproduce the above copyright notice, this list of conditions and the following disclaimer in the documentation and/or other materials provided with the distribution.
+      3. Neither the name of the copyright holder nor the names of its contributors may be used to endorse or promote products derived from this software without specific prior written permission.
+      THIS SOFTWARE IS PROVIDED BY THE COPYRIGHT HOLDERS AND CONTRIBUTORS "AS IS" AND ANY EXPRESS OR IMPLIED WARRANTIES, INCLUDING, BUT NOT LIMITED TO, THE IMPLIED WARRANTIES OF MERCHANTABILITY AND FITNESS FOR A PARTICULAR PURPOSE ARE DISCLAIMED.
+      IN NO EVENT SHALL THE COPYRIGHT HOLDER OR CONTRIBUTORS BE LIABLE FOR ANY DIRECT, INDIRECT, INCIDENTAL, SPECIAL, EXEMPLARY, OR CONSEQUENTIAL DAMAGES (INCLUDING, BUT NOT LIMITED TO, PROCUREMENT OF SUBSTITUTE GOODS OR SERVICES; LOSS OF USE, DATA, OR PROFITS; OR BUSINESS INTERRUPTION) HOWEVER CAUSED AND ON ANY THEORY OF LIABILITY, WHETHER IN CONTRACT, STRICT LIABILITY, OR TORT (INCLUDING NEGLIGENCE OR OTHERWISE) ARISING IN ANY WAY OUT OF THE USE OF THIS SOFTWARE, EVEN IF ADVISED OF THE POSSIBILITY OF SUCH DAMAGE.
+    -->
+    <!-- It has been modified to include the robot_name as a prefix to the links -->
+    <!-- It currently does not allow for simulation in either Gazebo (formerly Ignition) or Gazebo Class -->
+    <xacro:include filename="$(find interbotix_xslocobot_descriptions)/urdf/create3/bumper.urdf.xacro" />
+    <xacro:include filename="$(find interbotix_xslocobot_descriptions)/urdf/create3/button.urdf.xacro" />
+    <xacro:include filename="$(find interbotix_xslocobot_descriptions)/urdf/create3/caster.urdf.xacro" />
+    <xacro:include filename="$(find interbotix_xslocobot_descriptions)/urdf/create3/common_properties.urdf.xacro"/>
+    <xacro:include filename="$(find interbotix_xslocobot_descriptions)/urdf/create3/sensors/cliff_sensor.urdf.xacro"/>
+    <xacro:include filename="$(find interbotix_xslocobot_descriptions)/urdf/create3/sensors/imu.urdf.xacro" />
+    <xacro:include filename="$(find interbotix_xslocobot_descriptions)/urdf/create3/sensors/ir_intensity.urdf.xacro" />
+    <xacro:include filename="$(find interbotix_xslocobot_descriptions)/urdf/create3/sensors/ir_opcode_receivers.urdf.xacro" />
+    <xacro:include filename="$(find interbotix_xslocobot_descriptions)/urdf/create3/sensors/optical_mouse.urdf.xacro"/>
+    <xacro:include filename="$(find interbotix_xslocobot_descriptions)/urdf/create3/wheel_with_wheeldrop.urdf.xacro" />
+    <!-- Gazebo version -->
+    <xacro:arg name="gazebo"                       default="classic" />
+    <!-- Mechanical properties -->
+    <xacro:property name="body_z_offset"           value="${-2.5*cm2m}" />
+    <xacro:property name="body_collision_z_offset" value="${1*cm2m}" />
+    <xacro:property name="body_mass"               value="2.300" />
+    <xacro:property name="body_radius"             value="${16.4*cm2m}" />
+    <xacro:property name="body_length"             value="${6*cm2m}" />
+    <xacro:if value="${'$(arg gazebo)' == 'ignition'}">
+      <xacro:property name="body_cog_x_offset"       value="${2.28*cm2m}" />
+    </xacro:if>
+    <xacro:if value="${'$(arg gazebo)' == 'classic'}">
+      <xacro:property name="body_cog_x_offset"       value="${0*cm2m}" />
+    </xacro:if>
+    <xacro:property name="bumper_mass"             value="0.1" />
+    <xacro:property name="bumper_offset_z"         value="${-2.5*cm2m}" />
+    <xacro:property name="bumper_inertial_x"       value="${8*cm2m}" />
+    <xacro:property name="bumper_inertial_z"       value="${2*cm2m}"/>
+    <xacro:property name="wheel_height"            value="${-2.75*cm2m}" />
+    <xacro:property name="distance_between_wheels" value="${23.3*cm2m}" />
+    <xacro:property name="caster_position_x"       value="${12.5*cm2m}" />
+    <xacro:if value="${'$(arg gazebo)' == 'ignition'}">
+      <xacro:property name="caster_position_z"       value="${-5.03*cm2m}" />
+    </xacro:if>
+    <xacro:if value="${'$(arg gazebo)' == 'classic'}">
+      <xacro:property name="caster_position_z"       value="${-5.2*cm2m}" />
+    </xacro:if>
+    <xacro:property name="wheel_drop_offset_z"     value="${3.5*mm2m}"/>
+    <xacro:property name="wheel_drop_z"            value="${wheel_height + wheel_drop_offset_z}"/>
+    <xacro:property name="base_link_z_offset"     value="${6.42*cm2m}"/>
+    <joint name="base_joint" type="fixed">
       <origin rpy="0 0 0" xyz="0 0 0"/>
-      <geometry>
-        <mesh filename="package://interbotix_xslocobot_descriptions/meshes/locobot_meshes/locobot_wheel.dae"/>
-      </geometry>
-    </visual>
-    <collision>
-      <geometry>
-        <cylinder length="0.0206" radius="0.0352"/>
-      </geometry>
-        <origin rpy="0 0 0" xyz="0 0 0"/>
-    </collision>
-    <inertial>
-      <origin xyz="0 0 0"/>
-      <mass value="0.01"/>
-      <inertia ixx="0.001" ixy="0.0" ixz="0.0" iyy="0.001" iyz="0.0" izz="0.001"/>
-    </inertial>
-  </link>
-  <joint name="wheel_right_joint" type="continuous">
-    <axis xyz="0 0 1"/>
-    <origin rpy="-1.57079632679 0 0" xyz="0.00 -0.115 0.0250"/>
-    <parent link="$(arg robot_name)/base_link"/>
-    <child link="$(arg robot_name)/wheel_right_link"/>
-  </joint>
-  <transmission name="trans_wheel_right_joint">
-    <type>transmission_interface/SimpleTransmission</type>
-    <joint name="wheel_right_joint">
-      <hardwareInterface>hardware_interface/EffortJointInterface</hardwareInterface>
-    </joint>
-    <actuator name="wheel_right_joint_motor">
-      <mechanicalReduction>1</mechanicalReduction>
-    </actuator>
-  </transmission>
-  <link name="$(arg robot_name)/wheel_right_link">
-    <visual>
-      <origin rpy="0 0 0" xyz="0 0 0"/>
-      <geometry>
-        <mesh filename="package://interbotix_xslocobot_descriptions/meshes/locobot_meshes/locobot_wheel.dae"/>
-      </geometry>
-    </visual>
-    <collision>
-      <origin rpy="0 0 0" xyz="0 0 0"/>
-      <geometry>
-        <cylinder length="0.0206" radius="0.0350"/>
-      </geometry>
-    </collision>
-    <inertial>
-      <origin xyz="0 0 0"/>
-      <mass value="0.01"/>
-      <inertia ixx="0.001" ixy="0.0" ixz="0.0" iyy="0.001" iyz="0.0" izz="0.001"/>
-    </inertial>
-  </link>
-  <joint name="caster_front_joint" type="fixed">
-    <origin rpy="-1.57079632679 0 0" xyz="0.115 0.0 0.007"/>
-    <parent link="$(arg robot_name)/base_link"/>
-    <child link="$(arg robot_name)/caster_front_link"/>
-  </joint>
-  <link name="$(arg robot_name)/caster_front_link">
-    <collision>
-      <origin rpy="0 0 0" xyz="0 0 0"/>
-      <geometry>
-        <cylinder length="0.0176" radius="0.017"/>
-      </geometry>
-    </collision>
-    <inertial>
-      <origin xyz="0 0 0"/>
-      <mass value="0.01"/>
-      <inertia ixx="0.001" ixy="0.0" ixz="0.0" iyy="0.001" iyz="0.0" izz="0.001"/>
-    </inertial>
-  </link>
-  <joint name="caster_back_joint" type="fixed">
-    <origin rpy="-1.57079632679 0 0" xyz="-0.135 0.0 0.009"/>
-    <parent link="$(arg robot_name)/base_link"/>
-    <child link="$(arg robot_name)/caster_back_link"/>
-  </joint>
-  <link name="$(arg robot_name)/caster_back_link">
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