Commit message: [xslocobot_descriptions] Sim improvements
Small improvements to Gazebo configs and plugins. Other minor changes.

[skip ci]

File: interbotix_ros_xslocobots/interbotix_xslocobot_descriptions/urdf/arm_cradle.urdf.xacro (robot description, xacro)
@@ -30,4 +30,7 @@
      </link>
     </xacro:if>
+    <gazebo reference="arm_cradle">
+      <disableFixedJointLumping>true</disableFixedJointLumping>
+    </gazebo>
   </xacro:macro>
 </robot>

File: interbotix_ros_xslocobots/interbotix_xslocobot_descriptions/urdf/arms/mobile_arm.urdf.xacro (robot description, xacro)
@@ -130,7 +130,4 @@
       <disableFixedJointLumping>true</disableFixedJointLumping>
     </gazebo>
-    <gazebo reference="arm_cradle">
-      <disableFixedJointLumping>true</disableFixedJointLumping>
-    </gazebo>
   </xacro:macro>
 </robot>

File: interbotix_ros_xslocobots/interbotix_xslocobot_descriptions/urdf/arms/mobile_px100.urdf.xacro (robot description, xacro)
@@ -330,7 +330,5 @@
         <child link="$(arg robot_name)/right_finger_link"/>
         <dynamics friction="0.1"/>
-        <xacro:unless value="$(arg load_gazebo_configs)">
-          <mimic joint="left_finger" multiplier="-1" offset="0"/>
-        </xacro:unless>
+        <mimic joint="left_finger" multiplier="-1" offset="0"/>
       </joint>
       <transmission name="trans_right_finger">

File: interbotix_ros_xslocobots/interbotix_xslocobot_descriptions/urdf/arms/mobile_wx200.urdf.xacro (robot description, xacro)
@@ -367,7 +367,5 @@
         <child link="$(arg robot_name)/right_finger_link"/>
         <dynamics friction="0.1"/>
-        <xacro:unless value="$(arg load_gazebo_configs)">
-          <mimic joint="left_finger" multiplier="-1" offset="0"/>
-        </xacro:unless>
+        <mimic joint="left_finger" multiplier="-1" offset="0"/>
       </joint>
       <transmission name="trans_right_finger">

File: interbotix_ros_xslocobots/interbotix_xslocobot_descriptions/urdf/arms/mobile_wx250s.urdf.xacro (robot description, xacro)
@@ -404,7 +404,5 @@
         <child link="$(arg robot_name)/right_finger_link"/>
         <dynamics friction="0.1"/>
-        <xacro:unless value="$(arg load_gazebo_configs)">
-          <mimic joint="left_finger" multiplier="-1" offset="0"/>
-        </xacro:unless>
+        <mimic joint="left_finger" multiplier="-1" offset="0"/>
       </joint>
       <transmission name="trans_right_finger">

File: interbotix_ros_xslocobots/interbotix_xslocobot_descriptions/urdf/create3_version/locobot_create3.urdf.xacro (robot description, xacro)
@@ -210,5 +210,5 @@
       <commandTopic>cmd_vel</commandTopic>
       <odometryTopic>odom</odometryTopic>
-      <odometryFrame>odom</odometryFrame>
+      <odometryFrame>$(arg robot_name)/odom</odometryFrame>
       <robotBaseFrame>$(arg robot_name)/base_footprint</robotBaseFrame>
       <publishWheelJointState>true</publishWheelJointState>
@@ -224,5 +224,5 @@
       <update_rate>62</update_rate>
       <bodyName>$(arg robot_name)/base_link</bodyName>
-      <topicName>base/sim_ground_truth_pose</topicName>
+      <topicName>mobile_base/sim_ground_truth_pose</topicName>
       <namespace>/</namespace>
       <frameName>map</frameName>

File: interbotix_ros_xslocobots/interbotix_xslocobot_descriptions/urdf/kobuki_version/locobot_kobuki.urdf.xacro (robot description, xacro)
@@ -391,5 +391,5 @@
       <updateRate>100.0</updateRate>
       <bodyName>$(arg robot_name)/base_link</bodyName>
-      <topicName>base/absolute_position</topicName>
+      <topicName>mobile_base/absolute_position</topicName>
       <gaussianNoise>0</gaussianNoise>
       <frameName>map</frameName>

File: interbotix_ros_xslocobots/interbotix_xslocobot_descriptions/urdf/locobot.urdf.xacro (robot description, xacro)
@@ -9,5 +9,4 @@
   <xacro:arg name="show_gripper_fingers"  default="true"/>
   <xacro:arg name="external_urdf_loc"     default=""/>
-  <xacro:arg name="load_gazebo_configs"   default="false"/>
   <xacro:property name="arm_type"         value="$(arg arm_model)"/>
   <xacro:property name="base_type"        value="$(arg base_model)"/>
