Commit message: [xslocobot_descriptions] Match camera frame
Match the camera frame to the ones output by the realsense camera.

File: interbotix_ros_xslocobots/interbotix_xslocobot_descriptions/urdf/pan_and_tilt.urdf.xacro (robot description, xacro)
@@ -144,10 +144,10 @@
         link="${robot_name}/tilt_link"/>
       <child
-        link="${robot_name}/camera_link"/>
+        link="camera_${robot_name}_link"/>
     </joint>
     <gazebo reference="camera">
       <disableFixedJointLumping>true</disableFixedJointLumping>
     </gazebo>
-    <link name="${robot_name}/camera_link">
+    <link name="camera_${robot_name}_link">
       <visual>
         <origin
@@ -188,5 +188,5 @@
       </inertial>
     </link>
-    <gazebo reference="${robot_name}/camera_link">
+    <gazebo reference="camera_${robot_name}_link">
       <material>Gazebo/Grey</material>
       <self_collide>true</self_collide>
@@ -196,5 +196,5 @@
     <joint name="camera_depth_joint" type="fixed">
       <origin rpy="${-pi/2} 0 ${-pi/2}" xyz="0 0 0"/>
-      <parent link="${robot_name}/camera_link"/>
+      <parent link="camera_${robot_name}_link"/>
       <child link="${robot_name}/camera_depth_link"/>
     </joint>
@@ -202,5 +202,5 @@
       <origin rpy="0 0 0" xyz="0 0 0"/>
     </link>
-    <gazebo reference="${robot_name}/camera_link">
+    <gazebo reference="camera_${robot_name}_link">
       <sensor name="camera_frame_sensor" type="depth">
         <always_on>true</always_on>
