Commit message: [xslocobot_descriptions] Refine URDF
Clean up TODOs in URDF and add small camera tower mesh.

File: interbotix_ros_xslocobots/interbotix_xslocobot_descriptions/urdf/arms/mobile_arm.urdf.xacro (robot description, xacro)
@@ -18,5 +18,5 @@
       <joint name="arm_stand_link_joint" type="fixed">
         <axis xyz="0 0 0"/>
-        <origin rpy="0 0 0" xyz="0.111126 0 0.0095"/> <!-- TODO -->
+        <origin rpy="0 0 0" xyz="0.092002 0 0.007763"/>
         <parent link="$(arg robot_name)/plate_link"/>
         <child link="$(arg robot_name)/arm_stand_link"/>
@@ -44,5 +44,5 @@
       <joint name="arm_base_link_joint" type="fixed">
         <axis xyz="0 0 0"/>
-        <origin rpy="0 0 0" xyz="0 0 0.0095"/> <!-- TODO -->
+        <origin rpy="0 0 0" xyz="0 0 0.023"/>
         <parent link="$(arg robot_name)/arm_stand_link"/>
         <child link="$(arg robot_name)/arm_base_link"/>

File: interbotix_ros_xslocobots/interbotix_xslocobot_descriptions/urdf/locobot.urdf.xacro (robot description, xacro)
@@ -57,5 +57,5 @@
   <xacro:if value="${base_type == 'create3'}">
     <xacro:plate>
-      <origin rpy="0 0 0" xyz="0 0 0.0934"/> <!-- TODO -->
+      <origin rpy="0 0 0" xyz="0 0 0.0934"/>
       <inertial>
         <origin rpy="0 0 0" xyz="-0.005869 0 4.67E-03"/>
@@ -77,5 +77,5 @@
       <xacro:if value="${base_type == 'create3'}">
         <xacro:arm_cradle>
-          <origin rpy="0 0 0" xyz="0.0215 0 0.1195"/> <!-- TODO -->
+          <origin rpy="0 0 0" xyz="0.037943 0 0.139"/>
         </xacro:arm_cradle>
       </xacro:if> <!-- base_type == 'create3' -->
@@ -90,5 +90,5 @@
   <xacro:if value="${base_type == 'create3'}">
     <xacro:battery>
-      <origin rpy="0 0 0" xyz="-0.01 0 0.0125"/> <!-- TODO -->
+      <origin rpy="0 0 0" xyz="-0.0345 0 0.010763"/>
     </xacro:battery>
   </xacro:if> <!-- base_type == 'create3' -->
@@ -119,9 +119,9 @@
     <xacro:if value="${camera_tower_size == 'large'}">
       <xacro:camera_tower>
-        <origin rpy="0 0 0" xyz="-0.023997 -0.000044 0.08823"/> <!-- TODO -->
+        <origin rpy="0 0 0" xyz="-0.048271 0 0.10087"/>
         <inertial>
-          <origin rpy="0 0 0" xyz="-0.0372211000 -0.0026114300 0.1744600000"/>
-          <mass value="2.366224"/>
-          <inertia ixx="0.0628500000" ixy="0.0002152000" ixz="0.0065630000" iyy="0.0546000000" iyz="-0.0004738000" izz="0.0179300000"/>
+          <origin rpy="0 0 0" xyz="-0.025958 -0.003319 0.205872"/>
+          <mass value="2.514064"/>
+          <inertia ixx="7.61E-02" ixy="1.47E-04" ixz="7.04E-03" iyy="6.71E-02" iyz="-9.41E-04" izz="1.95E-02"/>
         </inertial>
       </xacro:camera_tower>
@@ -129,9 +129,9 @@
     <xacro:if value="${camera_tower_size == 'small'}">
       <xacro:camera_tower>
-        <origin rpy="0 0 0" xyz="-0.023997 -0.000044 0.08823"/> <!-- TODO -->
+        <origin rpy="0 0 0" xyz="-0.048271 0 0.10087"/>
         <inertial>
-          <origin rpy="0 0 0" xyz="-0.0357703000 -0.0027068600 0.1560470000"/>
-          <mass value="2.282808"/>
-          <inertia ixx="0.0461600000" ixy="0.0002062000" ixz="0.0052560000" iyy="0.0384200000" iyz="-0.0003600000" izz="0.0169600000"/>
+          <origin rpy="0 0 0" xyz="-0.024689 -0.003432 0.185408"/>
+          <mass value="2.430647"/>
+          <inertia ixx="5.63E-02" ixy="1.37E-04" ixz="5.75E-03" iyy="4.78E-02" iyz="-7.70E-04" izz="1.86E-02"/>
         </inertial>
       </xacro:camera_tower>
@@ -154,10 +154,10 @@
     <xacro:if value="${camera_tower_size == 'large'}">
       <xacro:pan_and_tilt>
-        <origin rpy="0 0 0" xyz="0 0 0"/> <!-- TODO -->
+        <origin rpy="0 0 0" xyz="0.061228 0 0.462"/>
       </xacro:pan_and_tilt>
     </xacro:if> <!-- base_type == 'create3' && camera_tower_size == 'large' -->
     <xacro:if value="${camera_tower_size == 'small'}">
       <xacro:pan_and_tilt>
-        <origin rpy="0 0 0" xyz="0 0 0"/> <!-- TODO -->
+        <origin rpy="0 0 0" xyz="0.061228 0 0.402"/>
       </xacro:pan_and_tilt>
     </xacro:if> <!-- base_type == 'create3' && camera_tower_size == 'small' -->
@@ -180,10 +180,10 @@
       <xacro:if value="${camera_tower_size == 'large'}">
         <xacro:lidar>
-          <origin rpy="0 0 0" xyz="-0.074 0 0.44425"/> <!-- TODO -->
+          <origin rpy="0 0 0" xyz="-0.066095 0 0.462"/>
         </xacro:lidar>
       </xacro:if> <!-- base_type == 'create3' && camera_tower_size == 'large' -->
       <xacro:if value="${camera_tower_size == 'small'}">
         <xacro:lidar>
-          <origin rpy="0 0 0" xyz="-0.074 0 0.38425"/> <!-- TODO -->
+          <origin rpy="0 0 0" xyz="-0.066095 0 0.402"/>
         </xacro:lidar>
       </xacro:if> <!-- base_type == 'create3' && camera_tower_size == 'small' -->
