Commit message: [xslocobot_descriptions] Add mock system joints
Adds pan, tilt, and create 3 base joints to the fake system with initial
positions set to silence moveit unknown state warnings.

File: interbotix_ros_xslocobots/interbotix_xslocobot_descriptions/urdf/arms/arm_control.urdf.xacro (robot description, xacro)
@@ -102,4 +102,40 @@
       </xacro:if>
     </xacro:if>
+    <joint name="pan">
+      <command_interface name="position"/>
+      <state_interface name="position"/>
+      <param name="initial_position">0.0</param>  <!-- initial position for the GenericSystem -->
+    </joint>
+    <joint name="tilt">
+      <command_interface name="position"/>
+      <state_interface name="position"/>
+      <param name="initial_position">0.0</param>  <!-- initial position for the GenericSystem -->
+    </joint>
+    <xacro:if value="${base_type == 'create3'}">
+      <joint name="wheel_drop_left_joint">
+        <command_interface name="position"/>
+        <state_interface name="position"/>
+        <param name="initial_position">0.0</param>  <!-- initial position for the GenericSystem -->
+      </joint>
+      <joint name="wheel_drop_right_joint">
+        <command_interface name="position"/>
+        <state_interface name="position"/>
+        <param name="initial_position">0.0</param>  <!-- initial position for the GenericSystem -->
+      </joint>
+      <joint name="left_wheel_joint">
+        <command_interface name="position"/>
+        <command_interface name="velocity"/>
+        <state_interface name="position"/>
+        <state_interface name="velocity"/>
+        <param name="initial_position">0.0</param>  <!-- initial position for the GenericSystem -->
+      </joint>
+      <joint name="right_wheel_joint">
+        <command_interface name="position"/>
+        <command_interface name="velocity"/>
+        <state_interface name="position"/>
+        <state_interface name="velocity"/>
+        <param name="initial_position">0.0</param>  <!-- initial position for the GenericSystem -->
+      </joint>
+    </xacro:if> <!-- $(base_type) == 'create3' -->
   </ros2_control>
 </robot>

Commit message: [xslocobot_descriptions] Add controllers condition
Adds the requirement that the hardware_type is set to fake to load some
joint interfaces.

File: interbotix_ros_xslocobots/interbotix_xslocobot_descriptions/urdf/arms/arm_control.urdf.xacro (robot description, xacro)
@@ -102,40 +102,42 @@
       </xacro:if>
     </xacro:if>
-    <joint name="pan">
-      <command_interface name="position"/>
-      <state_interface name="position"/>
-      <param name="initial_position">0.0</param>  <!-- initial position for the GenericSystem -->
-    </joint>
-    <joint name="tilt">
-      <command_interface name="position"/>
-      <state_interface name="position"/>
-      <param name="initial_position">0.0</param>  <!-- initial position for the GenericSystem -->
-    </joint>
-    <xacro:if value="${base_type == 'create3'}">
-      <joint name="wheel_drop_left_joint">
+    <xacro:if value="${hardware_type == 'fake'}">
+      <joint name="pan">
         <command_interface name="position"/>
         <state_interface name="position"/>
         <param name="initial_position">0.0</param>  <!-- initial position for the GenericSystem -->
       </joint>
-      <joint name="wheel_drop_right_joint">
+      <joint name="tilt">
         <command_interface name="position"/>
         <state_interface name="position"/>
         <param name="initial_position">0.0</param>  <!-- initial position for the GenericSystem -->
       </joint>
-      <joint name="left_wheel_joint">
-        <command_interface name="position"/>
-        <command_interface name="velocity"/>
-        <state_interface name="position"/>
-        <state_interface name="velocity"/>
-        <param name="initial_position">0.0</param>  <!-- initial position for the GenericSystem -->
-      </joint>
-      <joint name="right_wheel_joint">
-        <command_interface name="position"/>
-        <command_interface name="velocity"/>
-        <state_interface name="position"/>
-        <state_interface name="velocity"/>
-        <param name="initial_position">0.0</param>  <!-- initial position for the GenericSystem -->
-      </joint>
-    </xacro:if> <!-- $(base_type) == 'create3' -->
+      <xacro:if value="${base_type == 'create3'}">
+        <joint name="wheel_drop_left_joint">
+          <command_interface name="position"/>
+          <state_interface name="position"/>
+          <param name="initial_position">0.0</param>  <!-- initial position for the GenericSystem -->
+        </joint>
+        <joint name="wheel_drop_right_joint">
+          <command_interface name="position"/>
+          <state_interface name="position"/>
+          <param name="initial_position">0.0</param>  <!-- initial position for the GenericSystem -->
+        </joint>
+        <joint name="left_wheel_joint">
+          <command_interface name="position"/>
+          <command_interface name="velocity"/>
+          <state_interface name="position"/>
+          <state_interface name="velocity"/>
+          <param name="initial_position">0.0</param>  <!-- initial position for the GenericSystem -->
+        </joint>
+        <joint name="right_wheel_joint">
+          <command_interface name="position"/>
+          <command_interface name="velocity"/>
+          <state_interface name="position"/>
+          <state_interface name="velocity"/>
+          <param name="initial_position">0.0</param>  <!-- initial position for the GenericSystem -->
+        </joint>
+      </xacro:if> <!-- base_type == 'create3' -->
+    </xacro:if> <!-- hardware_type == 'gz_classic' -->
   </ros2_control>
 </robot>
