Commit message: [xslocobot_descriptions] Consider loading gz conf
Adds the load_gazebo_configs launch arg to the description launch file.
Uses that arg to build the xacro. Set right_finger joint to only mimic
left_finger if not using gazebo configs.

File: interbotix_ros_xslocobots/interbotix_xslocobot_descriptions/urdf/arms/mobile_px100.urdf.xacro (robot description, xacro)
@@ -330,5 +330,7 @@
         <child link="$(arg robot_name)/right_finger_link"/>
         <dynamics friction="0.1"/>
-        <mimic joint="left_finger" multiplier="-1" offset="0"/>
+        <xacro:unless value="$(arg load_gazebo_configs)">
+          <mimic joint="left_finger" multiplier="-1" offset="0"/>
+        </xacro:unless>
       </joint>
       <transmission name="trans_right_finger">

File: interbotix_ros_xslocobots/interbotix_xslocobot_descriptions/urdf/arms/mobile_wx200.urdf.xacro (robot description, xacro)
@@ -367,5 +367,7 @@
         <child link="$(arg robot_name)/right_finger_link"/>
         <dynamics friction="0.1"/>
-        <mimic joint="left_finger" multiplier="-1" offset="0"/>
+        <xacro:unless value="$(arg load_gazebo_configs)">
+          <mimic joint="left_finger" multiplier="-1" offset="0"/>
+        </xacro:unless>
       </joint>
       <transmission name="trans_right_finger">

File: interbotix_ros_xslocobots/interbotix_xslocobot_descriptions/urdf/arms/mobile_wx250s.urdf.xacro (robot description, xacro)
@@ -404,5 +404,7 @@
         <child link="$(arg robot_name)/right_finger_link"/>
         <dynamics friction="0.1"/>
-        <mimic joint="left_finger" multiplier="-1" offset="0"/>
+        <xacro:unless value="$(arg load_gazebo_configs)">
+          <mimic joint="left_finger" multiplier="-1" offset="0"/>
+        </xacro:unless>
       </joint>
       <transmission name="trans_right_finger">

File: interbotix_ros_xslocobots/interbotix_xslocobot_descriptions/urdf/locobot.urdf.xacro (robot description, xacro)
@@ -9,4 +9,5 @@
   <xacro:arg name="show_gripper_fingers"  default="true"/>
   <xacro:arg name="external_urdf_loc"     default=""/>
+  <xacro:arg name="load_gazebo_configs"   default="false"/>
   <xacro:property name="arm_type"         value="$(arg arm_model)"/>
   <xacro:property name="base_type"        value="$(arg base_model)"/>
