Commit message: [xslocobot_descriptions] Remove unused links
Removes base_footprint and the unused base_joint. Changes the show_lidar
argument to use_lidar.

File: interbotix_ros_xslocobots/interbotix_xslocobot_descriptions/urdf/create3_version/locobot_create3.urdf.xacro (robot description, xacro)
@@ -53,9 +53,4 @@
     <xacro:property name="wheel_drop_z"            value="${wheel_height + wheel_drop_offset_z}"/>
     <xacro:property name="base_link_z_offset"     value="${6.42*cm2m}"/>
-    <joint name="base_joint" type="fixed">
-      <origin rpy="0 0 0" xyz="0 0 0"/>
-      <parent link="${robot_name}/base_footprint"/>
-      <child link="${robot_name}/base_link"/>
-    </joint>
     <!-- Docking properties -->
     <xacro:property name="robot_model_name" value="create3"/>

File: interbotix_ros_xslocobots/interbotix_xslocobot_descriptions/urdf/locobot.urdf.xacro (robot description, xacro)
@@ -5,5 +5,5 @@
   <xacro:arg name="robot_name"            default=""/>
   <xacro:arg name="base_model"            default=""/>
-  <xacro:arg name="show_lidar"            default="true"/>
+  <xacro:arg name="use_lidar"             default="true"/>
   <xacro:arg name="show_ar_tag"           default="true"/>
   <xacro:arg name="show_gripper_bar"      default="true"/>
@@ -30,5 +30,4 @@
   <xacro:include filename="$(find interbotix_xslocobot_descriptions)/urdf/camera_tower.urdf.xacro" />
   <xacro:include filename="$(find interbotix_xslocobot_descriptions)/urdf/pan_and_tilt.urdf.xacro" />
-  <link name="${robot_name}/base_footprint"/>
   <xacro:if value="${arm_type == 'mobile_wx250s'}">
     <xacro:property name="camera_tower_size" value="large"/>
@@ -241,5 +240,5 @@
   </xacro:if> <!-- base_type == 'create3' -->
   <!-- ********************************** Lidar **********************************  -->
-  <xacro:if value="$(arg show_lidar)">
+  <xacro:if value="$(arg use_lidar)">
     <xacro:if value="${base_type == 'kobuki'}">
       <xacro:if value="${camera_tower_size == 'large'}">
@@ -274,4 +273,4 @@
       </xacro:if> <!-- base_type == 'create3' && camera_tower_size == 'small' -->
     </xacro:if> <!-- base_type == 'create3' -->
-  </xacro:if> <!-- show_lidar -->
+  </xacro:if> <!-- use_lidar -->
 </robot>
