Commit message: [xslocobot_descriptions] Configure sensor plugins
Configures the Create 3 sensor plugins. This change adds namespaces,
changes sensor names to valid ones, and removes unused simulated
sensors.

File: interbotix_ros_xslocobots/interbotix_xslocobot_descriptions/urdf/create3_version/bumper.urdf.xacro (robot description, xacro)
@@ -51,5 +51,5 @@
         <plugin name="${name}_plugin" filename="libgazebo_ros_create_bumper.so">
           <ros>
-            <namespace>/</namespace>
+            <namespace>/${robot_name}</namespace>
             <remapping>~/out:=_internal/bumper/event</remapping>
           </ros>

File: interbotix_ros_xslocobots/interbotix_xslocobot_descriptions/urdf/create3_version/dock/ir_emitter.urdf.xacro (robot description, xacro)
@@ -8,4 +8,5 @@
                                          min_range:=${7*cm2m}
                                          visualize:=false" >
+    <xacro:property name="sensor_name" value="${robot_name}_${name}" />
     <!-- Physical link properties -->
     <xacro:property name="mass" value="0.15" />
@@ -23,7 +24,7 @@
     <!-- This ray is not attached to any plugin, it is only used for aesthetic and debugging purposes
     only when the visualize flag is set. No need for high update rates. -->
-    <xacro:if value="${visualize}">
+    <!-- <xacro:if value="${visualize}">
       <gazebo reference="${robot_name}/${name}_link">
-        <xacro:ray_sensor sensor_name="${name}" gazebo="${gazebo}"
+        <xacro:ray_sensor sensor_name="${sensor_name}" gazebo="${gazebo}"
                       update_rate="${update_rate}" visualize="${visualize}"
                       h_samples="50" h_res="1.0" h_min_angle="-${aperture/2}" h_max_angle="${aperture/2}"
@@ -32,5 +33,5 @@
         </xacro:ray_sensor>
       </gazebo>
-    </xacro:if>
+    </xacro:if> -->
     <gazebo reference="${name}_joint" >
       <preserveFixedJoint>true</preserveFixedJoint>

File: interbotix_ros_xslocobots/interbotix_xslocobot_descriptions/urdf/create3_version/dock/standard_dock.urdf.xacro (robot description, xacro)
@@ -77,5 +77,5 @@
       <plugin name="gazebo_ros_p3d_dock" filename="libgazebo_ros_p3d.so">
         <ros>
-          <namespace>/</namespace>
+          <namespace>/${robot_name}</namespace>
           <remapping>odom:=sim_ground_truth_dock_pose</remapping>
         </ros>

File: interbotix_ros_xslocobots/interbotix_xslocobot_descriptions/urdf/create3_version/locobot_create3.urdf.xacro (robot description, xacro)
@@ -117,4 +117,9 @@
       <gazebo>
         <plugin name="gazebo_ros2_control" filename="libgazebo_ros2_control.so">
+          <ros>
+            <namespace>/$(arg robot_name)</namespace>
+          </ros>
+          <robot_param>robot_description</robot_param>
+          <robot_param_node>robot_state_publisher</robot_param_node>
           <parameters> $(find interbotix_xslocobot_sim)/config/create3_version/$(arg robot_model)_controllers.yaml </parameters>
         </plugin>
@@ -223,5 +228,5 @@
             <remapping>odom:=sim_ground_truth_pose</remapping>
           </ros>
-          <body_name>${robot_name}/base_footprint</body_name>
+          <body_name>${robot_name}/base_link</body_name>
           <frame_name>world</frame_name>
           <update_rate>62</update_rate>
@@ -235,5 +240,5 @@
         <plugin name="dock_status_publisher" filename="libgazebo_ros_create_docking_status.so">
           <ros>
-            <namespace>/</namespace>
+            <namespace>/${robot_name}</namespace>
             <remapping>~/out:=dock</remapping>
           </ros>

File: interbotix_ros_xslocobots/interbotix_xslocobot_descriptions/urdf/create3_version/sensors/cliff_sensor.urdf.xacro (robot description, xacro)
@@ -10,5 +10,5 @@
   <xacro:property name="max_range"           value="${15*cm2m}"/>
   <xacro:property name="samples"             value="${fov_deg/5}"/>
-  <xacro:property name="sensor_name"         value="${robot_name}/cliff_${name}"/>
+  <xacro:property name="sensor_name"         value="cliff_${name}"/>
   <xacro:property name="detection_threshold" value="${8*cm2m}"/>
   <joint name="${sensor_name}_joint" type="fixed">
@@ -27,5 +27,5 @@
       <plugin name="${sensor_name}" filename="libgazebo_ros_create_cliff_sensor.so">
         <ros>
-          <namespace>/</namespace>
+          <namespace>/${robot_name}</namespace>
           <remapping>~/out:=_internal/${sensor_name}/event</remapping>
         </ros>

File: interbotix_ros_xslocobots/interbotix_xslocobot_descriptions/urdf/create3_version/sensors/imu.urdf.xacro (robot description, xacro)
@@ -59,5 +59,5 @@
         <plugin name="${name}_plugin" filename="libgazebo_ros_create_imu.so">
           <ros>
-            <namespace>/</namespace>
+            <namespace>/$(arg robot_name)</namespace>
             <remapping>~/out:=imu</remapping>
           </ros>

File: interbotix_ros_xslocobots/interbotix_xslocobot_descriptions/urdf/create3_version/sensors/ir_intensity.urdf.xacro (robot description, xacro)
@@ -8,4 +8,5 @@
                        visualize:=false *origin" >
     <xacro:property name="link_name" value="${robot_name}/ir_intensity_${name}"/>
+    <xacro:property name="sensor_name" value="${robot_name}_ir_intensity_${name}"/>
     <joint name="${link_name}_joint" type="fixed">
       <xacro:insert_block name="origin" />
@@ -19,6 +20,6 @@
       <preserveFixedJoint>true</preserveFixedJoint>
     </gazebo>
-    <gazebo reference="${link_name}">
-      <xacro:ray_sensor sensor_name="${link_name}" gazebo="${gazebo}"
+    <!-- <gazebo reference="${link_name}">
+      <xacro:ray_sensor sensor_name="${sensor_name}" gazebo="${gazebo}"
                       update_rate="${update_rate}" visualize="${visualize}"
                       h_samples="5" h_res="1.0" h_min_angle="-${fov/2}" h_max_angle="${fov/2}"
@@ -27,10 +28,10 @@
           <plugin filename="libgazebo_ros_create_ir_intensity_sensor.so" name="${link_name}">
             <ros>
-              <namespace>/</namespace>
+              <namespace>/${robot_name}</namespace>
               <remapping>~/out:=_internal/${link_name}</remapping>
             </ros>
           </plugin>
       </xacro:ray_sensor>
-    </gazebo>
+    </gazebo> -->
   </xacro:macro>
 </robot>

File: interbotix_ros_xslocobots/interbotix_xslocobot_descriptions/urdf/create3_version/sensors/ir_opcode_receivers.urdf.xacro (robot description, xacro)
@@ -52,5 +52,5 @@
         <plugin name="${name}_plugin" filename="libgazebo_ros_create_ir_opcode.so">
           <ros>
-            <namespace>/</namespace>
+            <namespace>/${robot_name}</namespace>
             <remapping>~/out:=ir_opcode</remapping>
           </ros>

File: interbotix_ros_xslocobots/interbotix_xslocobot_descriptions/urdf/create3_version/sensors/optical_mouse.urdf.xacro (robot description, xacro)
@@ -14,5 +14,5 @@
         <plugin name="${name}_plugin" filename="libgazebo_ros_create_optical_mouse.so">
             <ros>
-              <namespace>/</namespace>
+              <namespace>/${robot_name}</namespace>
               <remapping>~/out:=${name}</remapping>
             </ros>

File: interbotix_ros_xslocobots/interbotix_xslocobot_descriptions/urdf/create3_version/wheel_drop.urdf.xacro (robot description, xacro)
@@ -44,5 +44,5 @@
       <plugin name="${robot_name}/${wd_link_name}_plugin" filename="libgazebo_ros_create_wheel_drop.so">
         <ros>
-          <namespace>/</namespace>
+          <namespace>/${robot_name}</namespace>
           <remapping>~/out:=_internal/wheel_drop/${name}_wheel/event</remapping>
         </ros>

File: interbotix_ros_xslocobots/interbotix_xslocobot_descriptions/urdf/pan_and_tilt.urdf.xacro (robot description, xacro)
@@ -219,4 +219,7 @@
         </camera>
         <plugin filename="libgazebo_ros_camera.so" name="camera_frame_controller">
+          <ros>
+            <namespace>/$(arg robot_name)</namespace>
+          </ros>
           <alwaysOn>true</alwaysOn>
           <updateRate>0.0</updateRate>
