Commit message: [descriptions] Fix front caster sagging

File: interbotix_ros_xslocobots/interbotix_xslocobot_descriptions/urdf/create3_version/bump_caster.urdf.xacro (robot description, xacro)
@@ -3,8 +3,8 @@
   <xacro:macro name="bump_caster" params="*origin">
     <joint name="bump_caster" type="fixed">
-        <axis xyz="0 0 0"/>
-        <xacro:insert_block name="origin"/>
-        <parent link="$(arg robot_name)/base_link"/>
-        <child link="$(arg robot_name)/bump_caster_link"/>
+      <axis xyz="0 0 0"/>
+      <xacro:insert_block name="origin"/>
+      <parent link="$(arg robot_name)/base_link"/>
+      <child link="$(arg robot_name)/bump_caster_link"/>
     </joint>
     <link name="$(arg robot_name)/bump_caster_link">
@@ -17,7 +17,7 @@
       </visual>
       <collision>
-        <origin rpy="0 0 0" xyz="0 0 0"/>
+        <origin rpy="0 ${pi/2} 0" xyz="0 0 0"/>
         <geometry>
-          <mesh filename="package://interbotix_xslocobot_descriptions/meshes/locobot_meshes/create3_version/bump_caster.stl"/>
+          <cylinder radius="0.009" length="0.02"/>
         </geometry>
       </collision>

File: interbotix_ros_xslocobots/interbotix_xslocobot_descriptions/urdf/create3_version/caster.urdf.xacro (robot description, xacro)
@@ -25,7 +25,4 @@
     <xacro:inertial_sphere mass="${mass}" radius="${radius}"/>
   </link>
-  <gazebo reference="${name}_joint">
-    <preserveFixedJoint>true</preserveFixedJoint>
-  </gazebo>
   <gazebo reference="${name}_link">
     <material>Gazebo/DarkGrey</material>

Commit message: [descriptions] Fix front caster sagging

File: interbotix_ros_xslocobots/interbotix_xslocobot_descriptions/urdf/create3_version/bump_caster.urdf.xacro (robot description, xacro)
@@ -3,8 +3,8 @@
   <xacro:macro name="bump_caster" params="*origin">
     <joint name="bump_caster" type="fixed">
-        <axis xyz="0 0 0"/>
-        <xacro:insert_block name="origin"/>
-        <parent link="${robot_name}/base_link"/>
-        <child link="${robot_name}/bump_caster_link"/>
+      <axis xyz="0 0 0"/>
+      <xacro:insert_block name="origin"/>
+      <parent link="$(arg robot_name)/base_link"/>
+      <child link="$(arg robot_name)/bump_caster_link"/>
     </joint>
     <link name="${robot_name}/bump_caster_link">
@@ -17,7 +17,7 @@
       </visual>
       <collision>
-        <origin rpy="0 0 0" xyz="0 0 0"/>
+        <origin rpy="0 ${pi/2} 0" xyz="0 0 0"/>
         <geometry>
-          <mesh filename="package://interbotix_xslocobot_descriptions/meshes/locobot_meshes/create3_version/bump_caster.stl"/>
+          <cylinder radius="0.009" length="0.02"/>
         </geometry>
       </collision>

File: interbotix_ros_xslocobots/interbotix_xslocobot_descriptions/urdf/create3_version/caster.urdf.xacro (robot description, xacro)
@@ -25,7 +25,4 @@
     <xacro:inertial_sphere mass="${mass}" radius="${radius}"/>
   </link>
-  <gazebo reference="${name}_joint">
-    <preserveFixedJoint>true</preserveFixedJoint>
-  </gazebo>
   <gazebo reference="${robot_name}/${name}_link">
     <material>Gazebo/DarkGrey</material>
