Commit message: [xslocobot_descriptions] Add missing kobuki link
Adds the base_footprint link to the locobot_kobuki xacro.

File: interbotix_ros_xslocobots/interbotix_xslocobot_descriptions/urdf/kobuki_version/locobot_kobuki.urdf.xacro (robot description, xacro)
@@ -38,4 +38,5 @@
     # POSSIBILITY OF SUCH DAMAGE.
   -->
+  <link name="${robot_name}/base_footprint">
   <joint name="base_joint" type="fixed">
     <origin

Commit message: [xslocobot_descriptions] Fix xacro formatting

File: interbotix_ros_xslocobots/interbotix_xslocobot_descriptions/urdf/kobuki_version/locobot_kobuki.urdf.xacro (robot description, xacro)
@@ -38,5 +38,5 @@
     # POSSIBILITY OF SUCH DAMAGE.
   -->
-  <link name="${robot_name}/base_footprint">
+  <link name="${robot_name}/base_footprint"/>
   <joint name="base_joint" type="fixed">
     <origin
